File: bbf-europower.brd (EAGLE design)
At the start: 16.5 x 53.3 mm, 13 parts, among them J1 CON_HEADER_2X05-PTH, J2 CON_HEADER_2X05-PTH

Commit message: almost there
Parts:
- removed JP2: M05X2PTH, SparkFun:AVR_ICSP
- added JP4, JP5: (no value), SparkFun:1X05
Connections:
- net GND: now also JP4.1, JP4.2, JP4.3, JP4.4, JP4.5; no longer JP2.10, JP2.2, JP2.4, JP2.6, JP2.8
- net VEE: now also JP5.1, JP5.2, JP5.3, JP5.4, JP5.5; no longer JP2.1, JP2.3, JP2.5, JP2.7, JP2.9
Routing:
- net VEE: track 21.8 -> 11.0 mm
Other:
- board size 16.5 x 53.3 mm -> 16.5 x 54.6 mm
Changed lines of the file:
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@@
 <board>
 <plain>
-<wire x1="14.605" y1="0" x2="16.51" y2="1.905" width="0" layer="20" curve="90"/>
-<wire x1="16.51" y1="1.905" x2="16.51" y2="51.435" width="0" layer="20"/>
+<wire x1="14.605" y1="-1.27" x2="16.51" y2="0.635" width="0" layer="20" curve="90"/>
+<wire x1="16.51" y1="0.635" x2="16.51" y2="51.435" width="0" layer="20"/>
 <wire x1="16.51" y1="51.435" x2="15.25" y2="53.33" width="0" layer="20" curve="90"/>
 <wire x1="15.25" y1="53.33" x2="1.895" y2="53.33" width="0" layer="20"/>
 <wire x1="1.895" y1="53.33" x2="0" y2="51.435" width="0" layer="20" curve="90"/>
-<wire x1="0" y1="51.435" x2="0" y2="1.905" width="0" layer="20"/>
-<wire x1="0" y1="1.905" x2="1.905" y2="0" width="0" layer="20" curve="90"/>
-<wire x1="1.905" y1="0" x2="14.605" y2="0" width="0" layer="20"/>
+<wire x1="0" y1="51.435" x2="0" y2="0.635" width="0" layer="20"/>
+<wire x1="0" y1="0.635" x2="1.905" y2="-1.27" width="0" layer="20" curve="90"/>
+<wire x1="1.905" y1="-1.27" x2="14.605" y2="-1.27" width="0" layer="20"/>
 <text x="5.3975" y="26.67" size="0.8128" layer="25" ratio="15">cc-by-sa</text>
 <text x="5.08" y="24.765" size="0.8128" layer="25" ratio="15">G. Johnson</text>
@@
 </autorouter>
 <elements>
-<element name="JP2" library="SparkFun" package="AVR_ICSP" value="M05X2PTH" x="8.255" y="3.175" smashed="yes" rot="R90"/>
 <element name="J1" library="tomatek" package="M2X5" value="CON_HEADER_2X05-PTH" x="8.255" y="30.48" smashed="yes" rot="R180"/>
 <element name="C1" library="resistor" package="E2-5" value="47u" x="9.525" y="43.18" smashed="yes" rot="R180"/>
@@
 <attribute name="VALUE" x="1.905" y="48.26" size="1.27" layer="27"/>
 </element>
+<element name="JP4" library="SparkFun" package="1X05" value="" x="3.175" y="4.445" smashed="yes">
+<attribute name="VALUE" x="1.905" y="1.27" size="1.27" layer="27"/>
+</element>
+<element name="JP5" library="SparkFun" package="1X05" value="" x="3.175" y="0.635" smashed="yes">
+<attribute name="VALUE" x="1.905" y="-2.54" size="1.27" layer="27"/>
+</element>
 </elements>
 <signals>
 <signal name="GND">
-<contactref element="JP2" pad="8"/>
-<contactref element="JP2" pad="6"/>
-<contactref element="JP2" pad="4"/>
-<contactref element="JP2" pad="2"/>
-<contactref element="JP2" pad="10"/>
 <polygon width="0.254" layer="16" isolate="0.3048">
-<vertex x="14.605" y="0" curve="90"/>
-<vertex x="16.51" y="1.905"/>
+<vertex x="14.605" y="-1.27" curve="90"/>
+<vertex x="16.51" y="0.635"/>
 <vertex x="16.51" y="52.07" curve="90"/>
 <vertex x="15.24" y="53.34"/>
 <vertex x="1.905" y="53.34" curve="90"/>
 <vertex x="0" y="51.435"/>
-<vertex x="0" y="1.905" curve="90"/>
-<vertex x="1.905" y="0"/>
+<vertex x="0" y="0.635" curve="90"/>
+<vertex x="1.905" y="-1.27"/>
 </polygon>
 <contactref element="J1" pad="7"/>
@@
 <contactref element="J2" pad="4"/>
 <polygon width="0.254" layer="1" isolate="0.3048">
-<vertex x="14.605" y="0" curve="90"/>
-<vertex x="16.51" y="1.905"/>
+<vertex x="14.605" y="-1.27" curve="90"/>
+<vertex x="16.51" y="0.635"/>
 <vertex x="16.51" y="52.07" curve="90"/>
 <vertex x="15.24" y="53.34"/>
 <vertex x="1.905" y="53.34" curve="90"/>
 <vertex x="0" y="51.435"/>
-<vertex x="0" y="1.905" curve="90"/>
-<vertex x="1.905" y="0"/>
+<vertex x="0" y="0.635" curve="90"/>
+<vertex x="1.905" y="-1.27"/>
 </polygon>
 <contactref element="JP3" pad="1"/>
@@
 <contactref element="JP3" pad="3"/>
 <contactref element="JP3" pad="4"/>
+<contactref element="JP4" pad="5"/>
+<contactref element="JP4" pad="1"/>
+<contactref element="JP4" pad="2"/>
+<contactref element="JP4" pad="3"/>
+<contactref element="JP4" pad="4"/>
+<wire x1="10.795" y1="47.625" x2="13.335" y2="47.625" width="0" layer="19" extent="1-1"/>
+<wire x1="8.255" y1="47.625" x2="10.795" y2="47.625" width="0" layer="19" extent="1-1"/>
+<wire x1="5.715" y1="47.625" x2="8.255" y2="47.625" width="0" layer="19" extent="1-1"/>
+<wire x1="3.175" y1="47.625" x2="5.715" y2="47.625" width="0" layer="19" extent="1-1"/>
+<wire x1="8.509" y1="43.18" x2="8.255" y2="47.625" width="0" layer="19" extent="1-1"/>
 <wire x1="2.54" y1="39.37" x2="8.509" y2="43.18" width="0" layer="19" extent="1-1"/>
 <wire x1="5.715" y1="31.75" x2="2.54" y2="39.37" width="0" layer="19" extent="1-1"/>
@@
 <wire x1="5.715" y1="4.445" x2="8.255" y2="4.445" width="0" layer="19" extent="1-1"/>
 <wire x1="3.175" y1="4.445" x2="5.715" y2="4.445" width="0" layer="19" extent="1-1"/>
-<wire x1="13.335" y1="47.625" x2="10.795" y2="4.445" width="0" layer="19" extent="1-1"/>
-<wire x1="10.795" y1="47.625" x2="13.335" y2="47.625" width="0" layer="19" extent="1-1"/>
-<wire x1="8.255" y1="47.625" x2="10.795" y2="47.625" width="0" layer="19" extent="1-1"/>
-<wire x1="5.715" y1="47.625" x2="8.255" y2="47.625" width="0" layer="19" extent="1-1"/>
-<wire x1="3.175" y1="47.625" x2="5.715" y2="47.625" width="0" layer="19" extent="1-1"/>
 </signal>
 <signal name="VCC">
@@
 </signal>
 <signal name="VEE">
-<contactref element="JP2" pad="7"/>
-<contactref element="JP2" pad="5"/>
-<contactref element="JP2" pad="3"/>
-<contactref element="JP2" pad="1"/>
-<contactref element="JP2" pad="9"/>
-<wire x1="3.175" y1="1.905" x2="5.715" y2="1.905" width="0.8128" layer="1"/>
-<wire x1="5.715" y1="1.905" x2="8.255" y2="1.905" width="0.8128" layer="1"/>
-<wire x1="8.255" y1="1.905" x2="10.795" y2="1.905" width="0.8128" layer="1"/>
-<wire x1="10.795" y1="1.905" x2="13.335" y2="1.905" width="0.8128" layer="1"/>
 <contactref element="C2" pad="-"/>
 <contactref element="L2" pad="2"/>
@@
 <wire x1="1.27" y1="6.7945" x2="1.27" y2="3.175" width="1.016" layer="1"/>
 <wire x1="1.27" y1="3.175" x2="2.54" y2="1.905" width="1.016" layer="1"/>
-<wire x1="2.54" y1="1.905" x2="3.175" y2="1.905" width="1.016" layer="1"/>
 <wire x1="2.54" y1="8.0645" x2="3.3655" y2="8.89" width="1.016" layer="1"/>
 <wire x1="3.3655" y1="8.89" x2="5.969" y2="8.89" width="1.016" layer="1"/>
+<contactref element="JP5" pad="1"/>
+<contactref element="JP5" pad="5"/>
+<contactref element="JP5" pad="2"/>
+<contactref element="JP5" pad="3"/>
+<contactref element="JP5" pad="4"/>
+<wire x1="5.715" y1="0.635" x2="3.175" y2="0.635" width="0" layer="19" extent="1-1"/>
+<wire x1="8.255" y1="0.635" x2="5.715" y2="0.635" width="0" layer="19" extent="1-1"/>
+<wire x1="10.795" y1="0.635" x2="8.255" y2="0.635" width="0" layer="19" extent="1-1"/>
+<wire x1="13.335" y1="0.635" x2="10.795" y2="0.635" width="0" layer="19" extent="1-1"/>
+<wire x1="2.54" y1="1.905" x2="3.175" y2="0.635" width="0" layer="19" extent="1-1"/>
 </signal>
 <signal name="+12V">
