File: bbf-eurojacks.brd (EAGLE design)
At the start: 16.5 x 54.6 mm, 9 parts, among them J1 1502_03SLOTTED, J2 1502_03SLOTTED, J3 1502_03SLOTTED, J4 1502_03SLOTTED

Commit message: update names on boards and schematics
Other:
- board text added: "Émilie Gillet"
- board text removed: "Olivier Gillet"
Changed lines of the file:
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@@
 <wire x1="8.255" y1="6.985" x2="20.955" y2="6.985" width="0" layer="20"/>
 <text x="8.255" y="45.085" size="0.8128" layer="25" ratio="15" rot="R90">cc-by-sa</text>
-<text x="9.525" y="45.085" size="0.8128" layer="25" ratio="15" rot="R90">Olivier Gillet</text>
+<text x="9.525" y="45.085" size="0.8128" layer="25" ratio="15" rot="R90">Émilie Gillet</text>
 </plain>
 <attributes>
