File: bbf-pots.brd (EAGLE design)
At the start: 16.6 x 54.6 mm, 8 parts

Commit message: update names on boards and schematics
Other:
- board text added: "Émilie Gillet"
- board text removed: "Olivier Gillet"
Changed lines of the file:
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@@
 <text x="17.78" y="35.56" size="1.016" layer="25" ratio="15">B</text>
 <text x="12.065" y="53.975" size="0.8128" layer="25" ratio="15">cc-by-sa</text>
-<text x="12.065" y="52.705" size="0.7112" layer="25" ratio="15">Olivier Gillet</text>
+<text x="12.065" y="52.705" size="0.7112" layer="25" ratio="15">Émilie Gillet</text>
 </plain>
 <attributes>
